Commit message: Changed the simulation world
Modified the simulation world such that it resembles more what the
competition will be like. Elevated the hokuyo sensor to avoid it sensing
the wheels.

File: mybot_ws/src/mybot_description/urdf/mybot.xacro (robot description, xacro)
@@ -166,5 +166,5 @@
   <joint name="hokuyo_joint" type="fixed">
     <axis xyz="0 1 0" />
-    <origin xyz=".15 0 .1" rpy="0 0 0"/>
+    <origin xyz=".15 0 .2" rpy="0 0 0"/>
     <parent link="chassis"/>
     <child link="hokuyo"/>

Commit message: Made a new branch

File: mybot_ws/src/mybot_description/urdf/mybot.xacro (robot description, xacro)
@@ -76,5 +76,5 @@
     <!--origin xyz="0.1 0.13 0.1" rpy="0 1.5707 1.5707"/-->
     <collision name="collision">
-      <origin xyz="0 0 0" rpy="0 1.5707 1.5707"/>
+      <origin xyz="0.1 0.13 0.1" rpy="0 1.5707 1.5707"/>
       <geometry>
         <cylinder radius="0.1" length="0.05"/>
@@ -99,5 +99,5 @@
     <!--origin xyz="0.1 -0.13 0.1" rpy="0 1.5707 1.5707"/-->
     <collision name="collision">
-      <origin xyz="0 0 0" rpy="0 1.5707 1.5707"/>
+      <origin xyz="0.1 -0.13 0.1" rpy="0 1.5707 1.5707"/>
       <geometry>
         <cylinder radius="0.1" length="0.05"/>
